Commit message: 添加入口程序

File: src/sim/pybullet_env/assets/urdf/hexapod.urdf (robot description, URDF)
Before this commit: robot hexapod, 0 links, 0 joints
Links:
- added link LF_hip_link, mass 0.3; collision cylinder length=0.06 radius=0.02; visual cylinder length=0.06 radius=0.02
- added link LF_knee_link, mass 0.2; collision cylinder length=0.09 radius=0.02; visual cylinder length=0.09 radius=0.02
- added link LF_thigh_link, mass 0.25; collision cylinder length=0.08 radius=0.02; visual cylinder length=0.08 radius=0.02
- added link LM_hip_link, mass 0.3; collision cylinder length=0.06 radius=0.02; visual cylinder length=0.06 radius=0.02
- added link LM_knee_link, mass 0.2; collision cylinder length=0.09 radius=0.02; visual cylinder length=0.09 radius=0.02
- added link LM_thigh_link, mass 0.25; collision cylinder length=0.08 radius=0.02; visual cylinder length=0.08 radius=0.02
- added link LR_hip_link, mass 0.3; collision cylinder length=0.06 radius=0.02; visual cylinder length=0.06 radius=0.02
- added link LR_knee_link, mass 0.2; collision cylinder length=0.09 radius=0.02; visual cylinder length=0.09 radius=0.02
- added link LR_thigh_link, mass 0.25; collision cylinder length=0.08 radius=0.02; visual cylinder length=0.08 radius=0.02
- added link RF_hip_link, mass 0.3; collision cylinder length=0.06 radius=0.02; visual cylinder length=0.06 radius=0.02
- added link RF_knee_link, mass 0.2; collision cylinder length=0.09 radius=0.02; visual cylinder length=0.09 radius=0.02
- added link RF_thigh_link, mass 0.25; collision cylinder length=0.08 radius=0.02; visual cylinder length=0.08 radius=0.02
- added link RM_hip_link, mass 0.3; collision cylinder length=0.06 radius=0.02; visual cylinder length=0.06 radius=0.02
- added link RM_knee_link, mass 0.2; collision cylinder length=0.09 radius=0.02; visual cylinder length=0.09 radius=0.02
- added link RM_thigh_link, mass 0.25; collision cylinder length=0.08 radius=0.02; visual cylinder length=0.08 radius=0.02
- added link RR_hip_link, mass 0.3; collision cylinder length=0.06 radius=0.02; visual cylinder length=0.06 radius=0.02
- added link RR_knee_link, mass 0.2; collision cylinder length=0.09 radius=0.02; visual cylinder length=0.09 radius=0.02
- added link RR_thigh_link, mass 0.25; collision cylinder length=0.08 radius=0.02; visual cylinder length=0.08 radius=0.02
- added link base, mass 6.0; collision box size=0.35 0.25 0.08; visual box size=0.35 0.25 0.08
Joints:
- added joint LF_HIP: type revolute, parent base, child LF_hip_link, origin xyz=0.18 0.15 0.02 rpy=0 0 0, axis 0 0 1, limit lower=-1.0 upper=1.0 effort=5 velocity=4.0
- added joint LF_KNEE: type revolute, parent LF_thigh_link, child LF_knee_link, origin xyz=0.0 0.0 -0.04 rpy=0 0 0, axis 0 1 0, limit lower=-1.0 upper=1.0 effort=5 velocity=4.0
- added joint LF_THIGH: type revolute, parent LF_hip_link, child LF_thigh_link, origin xyz=0.03 0 0 rpy=0 0 0, axis 0 1 0, limit lower=-1.5 upper=1.5 effort=5 velocity=4.0
- added joint LM_HIP: type revolute, parent base, child LM_hip_link, origin xyz=0.0 0.15 0.02 rpy=0 0 0, axis 0 0 1, limit lower=-1.0 upper=1.0 effort=5 velocity=4.0
- added joint LM_KNEE: type revolute, parent LM_thigh_link, child LM_knee_link, origin xyz=0.0 0.0 -0.04 rpy=0 0 0, axis 0 1 0, limit lower=-1.0 upper=1.0 effort=5 velocity=4.0
- added joint LM_THIGH: type revolute, parent LM_hip_link, child LM_thigh_link, origin xyz=0.03 0 0 rpy=0 0 0, axis 0 1 0, limit lower=-1.5 upper=1.5 effort=5 velocity=4.0
- added joint LR_HIP: type revolute, parent base, child LR_hip_link, origin xyz=-0.18 0.15 0.02 rpy=0 0 0, axis 0 0 1, limit lower=-1.0 upper=1.0 effort=5 velocity=4.0
- added joint LR_KNEE: type revolute, parent LR_thigh_link, child LR_knee_link, origin xyz=0.0 0.0 -0.04 rpy=0 0 0, axis 0 1 0, limit lower=-1.0 upper=1.0 effort=5 velocity=4.0
- added joint LR_THIGH: type revolute, parent LR_hip_link, child LR_thigh_link, origin xyz=0.03 0 0 rpy=0 0 0, axis 0 1 0, limit lower=-1.5 upper=1.5 effort=5 velocity=4.0
- added joint RF_HIP: type revolute, parent base, child RF_hip_link, origin xyz=0.18 -0.15 0.02 rpy=0 0 0, axis 0 0 1, limit lower=-1.0 upper=1.0 effort=5 velocity=4.0
- added joint RF_KNEE: type revolute, parent RF_thigh_link, child RF_knee_link, origin xyz=0.0 0.0 -0.04 rpy=0 0 0, axis 0 1 0, limit lower=-1.0 upper=1.0 effort=5 velocity=4.0
- added joint RF_THIGH: type revolute, parent RF_hip_link, child RF_thigh_link, origin xyz=0.03 0 0 rpy=0 0 0, axis 0 1 0, limit lower=-1.5 upper=1.5 effort=5 velocity=4.0
- added joint RM_HIP: type revolute, parent base, child RM_hip_link, origin xyz=0.0 -0.15 0.02 rpy=0 0 0, axis 0 0 1, limit lower=-1.0 upper=1.0 effort=5 velocity=4.0
- added joint RM_KNEE: type revolute, parent RM_thigh_link, child RM_knee_link, origin xyz=0.0 0.0 -0.04 rpy=0 0 0, axis 0 1 0, limit lower=-1.0 upper=1.0 effort=5 velocity=4.0
- added joint RM_THIGH: type revolute, parent RM_hip_link, child RM_thigh_link, origin xyz=0.03 0 0 rpy=0 0 0, axis 0 1 0, limit lower=-1.5 upper=1.5 effort=5 velocity=4.0
- added joint RR_HIP: type revolute, parent base, child RR_hip_link, origin xyz=-0.18 -0.15 0.02 rpy=0 0 0, axis 0 0 1, limit lower=-1.0 upper=1.0 effort=5 velocity=4.0
- added joint RR_KNEE: type revolute, parent RR_thigh_link, child RR_knee_link, origin xyz=0.0 0.0 -0.04 rpy=0 0 0, axis 0 1 0, limit lower=-1.0 upper=1.0 effort=5 velocity=4.0
- added joint RR_THIGH: type revolute, parent RR_hip_link, child RR_thigh_link, origin xyz=0.03 0 0 rpy=0 0 0, axis 0 1 0, limit lower=-1.5 upper=1.5 effort=5 velocity=4.0
